File: flipperbrain-shield/flipperbrain-shield/flipperbrain-shield.kicad_pcb (KiCad board)
At the start: 2 copper layers, 68.6 x 53.3 mm, 10 parts, among them J1 Power, J2 Digital/PWM, J3 Analog, J4 Digital/PWM

Commit message: nc
Parts:
- moved R1 11.4 mm to (150.8, 87.3)
Connections:
- D1 pad 1: Net-(D1-K) -> GND
- D1 pad 2: A0 -> Net-(D1-A)
- R1 pad 1: Net-(D1-K) -> A0
- R1 pad 2: GND -> Net-(D1-A)

Commit message: nc
Parts:
- J3: footprint Connector_PinSocket_2.54mm:PinSocket_1x06_P2.54mm_Vertical -> Connector_PinHeader_2.54mm:PinHeader_1x06_P2.54mm_Vertical; moved to B.Cu
- moved D1 20.5 mm to (150.8, 72.1)
- turned J3 to -90 degrees
Changed lines of the file:
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@@
-    )
-  )
-  (footprint "Connector_PinSocket_2.54mm:PinSocket_1x06_P2.54mm_Vertical" locked (layer "F.Cu")
-    (at 150.8 97.46 90)
-    (descr "Through hole straight socket strip, 1x06, 2.54mm pitch, single row (from Kicad 4.0.7), script generated")
-    (tags "Through hole socket strip THT 1x06 2.54mm single row")
-    (property "Sheetfile" "flipperbrain-shield.kicad_sch")
-    (property "Sheetname" "")
-    (property "ki_description" "Generic connector, single row, 01x06, script generated (kicad-library-utils/schlib/autogen/connector/)")
-    (property "ki_keywords" "connector")
-    (attr through_hole)
-    (fp_text reference "J3" (at 0 -2.77 90) (layer "F.SilkS") hide
-        (effects (font (size 1 1) (thickness 0.15)))
-    )
-    (fp_text value "Analog" (at -3.81 6.35 180) (layer "F.Fab")
-        (effects (font (size 1 1) (thickness 0.15)))
-    )
-    (fp_text user "${REFERENCE}" (at -3.81 0 180) (layer "F.Fab")
-        (effects (font (size 1 1) (thickness 0.15)))
-    )
-    (fp_line (start -1.33 1.27) (end -1.33 14.03)
-      (stroke (width 0.12) (type solid)) (layer "F.SilkS"))
-    (fp_line (start -1.33 1.27) (end 1.33 1.27)
-      (stroke (width 0.12) (type solid)) (layer "F.SilkS"))
-    (fp_line (start -1.33 14.03) (end 1.33 14.03)
-      (stroke (width 0.12) (type solid)) (layer "F.SilkS"))
-    (fp_line (start 0 -1.33) (end 1.33 -1.33)
-      (stroke (width 0.12) (type solid)) (layer "F.SilkS"))
-    (fp_line (start 1.33 -1.33) (end 1.33 0)
-      (stroke (width 0.12) (type solid)) (layer "F.SilkS"))
-    (fp_line (start 1.33 1.27) (end 1.33 14.03)
-      (stroke (width 0.12) (type solid)) (layer "F.SilkS"))
-    (fp_line (start -1.8 -1.8) (end 1.75 -1.8)
-      (stroke (width 0.05) (type solid)) (layer "F.CrtYd"))
-    (fp_line (start -1.8 14.45) (end -1.8 -1.8)
-      (stroke (width 0.05) (type solid)) (layer "F.CrtYd"))
-    (fp_line (start 1.75 -1.8) (end 1.75 14.45)
-      (stroke (width 0.05) (type solid)) (layer "F.CrtYd"))
-    (fp_line (start 1.75 14.45) (end -1.8 14.45)
-      (stroke (width 0.05) (type solid)) (layer "F.CrtYd"))
-    (fp_line (start -1.27 -1.27) (end 0.635 -1.27)
-      (stroke (width 0.1) (type solid)) (layer "F.Fab"))
-    (fp_line (start -1.27 13.97) (end -1.27 -1.27)
-      (stroke (width 0.1) (type solid)) (layer "F.Fab"))
-    (fp_line (start 0.635 -1.27) (end 1.27 -0.635)
-      (stroke (width 0.1) (type solid)) (layer "F.Fab"))
-    (fp_line (start 1.27 -0.635) (end 1.27 13.97)
-      (stroke (width 0.1) (type solid)) (layer "F.Fab"))
-    (fp_line (start 1.27 13.97) (end -1.27 13.97)
-      (stroke (width 0.1) (type solid)) (layer "F.Fab"))
-    (pad "1" thru_hole rect locked (at 0 0 90) (size 1.7 1.7) (drill 1) (layers "*.Cu" "*.Mask")
-      (net 28 "A0") (pinfunction "Pin_1") (pintype "passive"))
-    (pad "2" thru_hole oval locked (at 0 2.54 90) (size 1.7 1.7) (drill 1) (layers "*.Cu" "*.Mask")
-      (net 5 "/A1") (pinfunction "Pin_2") (pintype "passive"))
-    (pad "3" thru_hole oval locked (at 0 5.08 90) (size 1.7 1.7) (drill 1) (layers "*.Cu" "*.Mask")
-      (net 6 "/A2") (pinfunction "Pin_3") (pintype "passive"))
-    (pad "4" thru_hole oval locked (at 0 7.62 90) (size 1.7 1.7) (drill 1) (layers "*.Cu" "*.Mask")
-      (net 7 "/A3") (pinfunction "Pin_4") (pintype "passive"))
-    (pad "5" thru_hole oval locked (at 0 10.16 90) (size 1.7 1.7) (drill 1) (layers "*.Cu" "*.Mask")
-      (net 8 "/SDA{slash}A4") (pinfunction "Pin_5") (pintype "passive"))
-    (pad "6" thru_hole oval locked (at 0 12.7 90) (size 1.7 1.7) (drill 1) (layers "*.Cu" "*.Mask")
-      (net 9 "/SCL{slash}A5") (pinfunction "Pin_6") (pintype "passive"))
-    (model "${KICAD7_3DMODEL_DIR}/Connector_PinSocket_2.54mm.3dshapes/PinSocket_1x06_P2.54mm_Vertical.wrl"
-      (offset (xyz 0 0 0))
-      (scale (xyz 1 1 1))
-      (rotate (xyz 0 0 0))
     )
   )
@@
   )
   (footprint "LED_THT:LED_D5.0mm" (layer "F.Cu")
-    (at 140.64 89.84 90)
+    (at 150.8 72.06 90)
     (descr "LED, diameter 5.0mm, 2 pins, http://cdn-reichelt.de/documents/datenblatt/A500/LL-504BC2E-009.pdf")
     (tags "LED diameter 5.0mm 2 pins")
@@
     (pad "" np_thru_hole circle locked (at 0 0) (size 3.2 3.2) (drill 3.2) (layers "*.Cu" "*.Mask"))
   )
+  (footprint "Connector_PinHeader_2.54mm:PinHeader_1x06_P2.54mm_Vertical" locked (layer "B.Cu")
+    (at 150.8 97.46 -90)
+    (descr "Through hole straight pin header, 1x06, 2.54mm pitch, single row")
+    (tags "Through hole pin header THT 1x06 2.54mm single row")
+    (property "Sheetfile" "flipperbrain-shield.kicad_sch")
+    (property "Sheetname" "")
+    (property "ki_description" "Generic connector, single row, 01x06, script generated (kicad-library-utils/schlib/autogen/connector/)")
+    (property "ki_keywords" "connector")
+    (attr through_hole)
+    (fp_text reference "J3" (at 0 2.33 90) (layer "B.SilkS")
+        (effects (font (size 1 1) (thickness 0.15)) (justify mirror))
+    )
+    (fp_text value "Analog" (at 0 -15.03 90) (layer "B.Fab")
+        (effects (font (size 1 1) (thickness 0.15)) (justify mirror))
+    )
+    (fp_text user "${REFERENCE}" (at 0 -6.35) (layer "B.Fab")
+        (effects (font (size 1 1) (thickness 0.15)) (justify mirror))
+    )
+    (fp_line (start -1.33 -14.03) (end 1.33 -14.03)
+      (stroke (width 0.12) (type solid)) (layer "B.SilkS"))
+    (fp_line (start -1.33 -1.27) (end -1.33 -14.03)
+      (stroke (width 0.12) (type solid)) (layer "B.SilkS"))
+    (fp_line (start -1.33 -1.27) (end 1.33 -1.27)
+      (stroke (width 0.12) (type solid)) (layer "B.SilkS"))
+    (fp_line (start -1.33 0) (end -1.33 1.33)
+      (stroke (width 0.12) (type solid)) (layer "B.SilkS"))
+    (fp_line (start -1.33 1.33) (end 0 1.33)
+      (stroke (width 0.12) (type solid)) (layer "B.SilkS"))
+    (fp_line (start 1.33 -1.27) (end 1.33 -14.03)
+      (stroke (width 0.12) (type solid)) (layer "B.SilkS"))
+    (fp_line (start -1.8 -14.5) (end 1.8 -14.5)
+      (stroke (width 0.05) (type solid)) (layer "B.CrtYd"))
+    (fp_line (start -1.8 1.8) (end -1.8 -14.5)
+      (stroke (width 0.05) (type solid)) (layer "B.CrtYd"))
+    (fp_line (start 1.8 -14.5) (end 1.8 1.8)
+      (stroke (width 0.05) (type solid)) (layer "B.CrtYd"))
+    (fp_line (start 1.8 1.8) (end -1.8 1.8)
+      (stroke (width 0.05) (type solid)) (layer "B.CrtYd"))
+    (fp_line (start -1.27 -13.97) (end -1.27 0.635)
+      (stroke (width 0.1) (type solid)) (layer "B.Fab"))
+    (fp_line (start -1.27 0.635) (end -0.635 1.27)
+      (stroke (width 0.1) (type solid)) (layer "B.Fab"))
+    (fp_line (start -0.635 1.27) (end 1.27 1.27)
+      (stroke (width 0.1) (type solid)) (layer "B.Fab"))
+    (fp_line (start 1.27 -13.97) (end -1.27 -13.97)
+      (stroke (width 0.1) (type solid)) (layer "B.Fab"))
+    (fp_line (start 1.27 1.27) (end 1.27 -13.97)
+      (stroke (width 0.1) (type solid)) (layer "B.Fab"))
+    (pad "1" thru_hole rect locked (at 0 0 270) (size 1.7 1.7) (drill 1) (layers "*.Cu" "*.Mask")
+      (net 28 "A0") (pinfunction "Pin_1") (pintype "passive"))
+    (pad "2" thru_hole oval locked (at 0 -2.54 270) (size 1.7 1.7) (drill 1) (layers "*.Cu" "*.Mask")
+      (net 5 "/A1") (pinfunction "Pin_2") (pintype "passive"))
+    (pad "3" thru_hole oval locked (at 0 -5.08 270) (size 1.7 1.7) (drill 1) (layers "*.Cu" "*.Mask")
+      (net 6 "/A2") (pinfunction "Pin_3") (pintype "passive"))
+    (pad "4" thru_hole oval locked (at 0 -7.62 270) (size 1.7 1.7) (drill 1) (layers "*.Cu" "*.Mask")
+      (net 7 "/A3") (pinfunction "Pin_4") (pintype "passive"))
+    (pad "5" thru_hole oval locked (at 0 -10.16 270) (size 1.7 1.7) (drill 1) (layers "*.Cu" "*.Mask")
+      (net 8 "/SDA{slash}A4") (pinfunction "Pin_5") (pintype "passive"))
+    (pad "6" thru_hole oval locked (at 0 -12.7 270) (size 1.7 1.7) (drill 1) (layers "*.Cu" "*.Mask")
+      (net 9 "/SCL{slash}A5") (pinfunction "Pin_6") (pintype "passive"))
+    (model "${KICAD6_3DMODEL_DIR}/Connector_PinHeader_2.54mm.3dshapes/PinHeader_1x06_P2.54mm_Vertical.wrl"
+      (offset (xyz 0 0 0))
+      (scale (xyz 1 1 1))
+      (rotate (xyz 0 0 0))
+    )
+  )
   (gr_line (start 98.095 96.825) (end 98.095 87.935)

Commit message: nc
Parts:
- removed J1: Power, Connector_PinSocket_2.54mm:PinSocket_1x08_P2.54mm_Vertical
- added J1-new1: Power, Connector_PinHeader_2.54mm:PinHeader_1x08_P2.54mm_Vertical, B.Cu at (127.9, 97.5)

Commit message: nc
Parts:
- renumbered J1-new1 to J1
Changed lines of the file:
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@@
   (net 27 "A0")
   (net 28 "Net-(D1-A)")
-  (net 29 "unconnected-(J1-new1-Pin_1-Pad1)")
+  (net 29 "unconnected-(J1-Pin_1-Pad1)")
   (footprint "Connector_PinSocket_2.54mm:PinSocket_1x10_P2.54mm_Vertical" locked (layer "F.Cu")
     (at 118.796 49.2 90)
@@
     (property "ki_keywords" "connector")
     (attr through_hole)
-    (fp_text reference "J1-new1" (at 0 2.33 90) (layer "B.SilkS")
+    (fp_text reference "J1" (at 0 2.33 90) (layer "B.SilkS")
         (effects (font (size 1 1) (thickness 0.15)) (justify mirror))
     )
@@
       (stroke (width 0.1) (type solid)) (layer "B.Fab"))
     (pad "1" thru_hole rect (at 0 0 270) (size 1.7 1.7) (drill 1) (layers "*.Cu" "*.Mask")
-      (net 29 "unconnected-(J1-new1-Pin_1-Pad1)") (pinfunction "Pin_1") (pintype "passive+no_connect"))
+      (net 29 "unconnected-(J1-Pin_1-Pad1)") (pinfunction "Pin_1") (pintype "passive+no_connect"))
     (pad "2" thru_hole oval (at 0 -2.54 270) (size 1.7 1.7) (drill 1) (layers "*.Cu" "*.Mask")
       (net 3 "/IOREF") (pinfunction "Pin_2") (pintype "passive"))

Commit message: nc
Parts:
- J2: footprint Connector_PinSocket_2.54mm:PinSocket_1x10_P2.54mm_Vertical -> Connector_PinHeader_2.54mm:PinHeader_1x10_P2.54mm_Vertical; moved to B.Cu
- turned J2 to -90 degrees
Changed lines of the file:
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@@
   (net 28 "Net-(D1-A)")
   (net 29 "unconnected-(J1-Pin_1-Pad1)")
-  (footprint "Connector_PinSocket_2.54mm:PinSocket_1x10_P2.54mm_Vertical" locked (layer "F.Cu")
-    (at 118.796 49.2 90)
-    (descr "Through hole straight socket strip, 1x10, 2.54mm pitch, single row (from Kicad 4.0.7), script generated")
-    (tags "Through hole socket strip THT 1x10 2.54mm single row")
-    (property "Sheetfile" "flipperbrain-shield.kicad_sch")
-    (property "Sheetname" "")
-    (property "ki_description" "Generic connector, single row, 01x10, script generated (kicad-library-utils/schlib/autogen/connector/)")
-    (property "ki_keywords" "connector")
-    (attr through_hole)
-    (fp_text reference "J2" (at 0 -2.77 90) (layer "F.SilkS") hide
-        (effects (font (size 1 1) (thickness 0.15)))
-    )
-    (fp_text value "Digital/PWM" (at 3.81 11.43 180) (layer "F.Fab")
-        (effects (font (size 1 1) (thickness 0.15)))
-    )
-    (fp_text user "${REFERENCE}" (at 3.81 0) (layer "F.Fab")
-        (effects (font (size 1 1) (thickness 0.15)))
-    )
-    (fp_line (start -1.33 1.27) (end -1.33 24.19)
-      (stroke (width 0.12) (type solid)) (layer "F.SilkS"))
-    (fp_line (start -1.33 1.27) (end 1.33 1.27)
-      (stroke (width 0.12) (type solid)) (layer "F.SilkS"))
-    (fp_line (start -1.33 24.19) (end 1.33 24.19)
-      (stroke (width 0.12) (type solid)) (layer "F.SilkS"))
-    (fp_line (start 0 -1.33) (end 1.33 -1.33)
-      (stroke (width 0.12) (type solid)) (layer "F.SilkS"))
-    (fp_line (start 1.33 -1.33) (end 1.33 0)
-      (stroke (width 0.12) (type solid)) (layer "F.SilkS"))
-    (fp_line (start 1.33 1.27) (end 1.33 24.19)
-      (stroke (width 0.12) (type solid)) (layer "F.SilkS"))
-    (fp_line (start -1.8 -1.8) (end 1.75 -1.8)
-      (stroke (width 0.05) (type solid)) (layer "F.CrtYd"))
-    (fp_line (start -1.8 24.6) (end -1.8 -1.8)
-      (stroke (width 0.05) (type solid)) (layer "F.CrtYd"))
-    (fp_line (start 1.75 -1.8) (end 1.75 24.6)
-      (stroke (width 0.05) (type solid)) (layer "F.CrtYd"))
-    (fp_line (start 1.75 24.6) (end -1.8 24.6)
-      (stroke (width 0.05) (type solid)) (layer "F.CrtYd"))
-    (fp_line (start -1.27 -1.27) (end 0.635 -1.27)
-      (stroke (width 0.1) (type solid)) (layer "F.Fab"))
-    (fp_line (start -1.27 24.13) (end -1.27 -1.27)
-      (stroke (width 0.1) (type solid)) (layer "F.Fab"))
-    (fp_line (start 0.635 -1.27) (end 1.27 -0.635)
-      (stroke (width 0.1) (type solid)) (layer "F.Fab"))
-    (fp_line (start 1.27 -0.635) (end 1.27 24.13)
-      (stroke (width 0.1) (type solid)) (layer "F.Fab"))
-    (fp_line (start 1.27 24.13) (end -1.27 24.13)
-      (stroke (width 0.1) (type solid)) (layer "F.Fab"))
-    (pad "1" thru_hole rect locked (at 0 0 90) (size 1.7 1.7) (drill 1) (layers "*.Cu" "*.Mask")
-      (net 8 "/SCL{slash}A5") (pinfunction "Pin_1") (pintype "passive"))
-    (pad "2" thru_hole oval locked (at 0 2.54 90) (size 1.7 1.7) (drill 1) (layers "*.Cu" "*.Mask")
-      (net 7 "/SDA{slash}A4") (pinfunction "Pin_2") (pintype "passive"))
-    (pad "3" thru_hole oval locked (at 0 5.08 90) (size 1.7 1.7) (drill 1) (layers "*.Cu" "*.Mask")
-      (net 11 "/AREF") (pinfunction "Pin_3") (pintype "passive"))
-    (pad "4" thru_hole oval locked (at 0 7.62 90) (size 1.7 1.7) (drill 1) (layers "*.Cu" "*.Mask")
-      (net 1 "GND") (pinfunction "Pin_4") (pintype "passive"))
-    (pad "5" thru_hole oval locked (at 0 10.16 90) (size 1.7 1.7) (drill 1) (layers "*.Cu" "*.Mask")
-      (net 9 "/13") (pinfunction "Pin_5") (pintype "passive"))
-    (pad "6" thru_hole oval locked (at 0 12.7 90) (size 1.7 1.7) (drill 1) (layers "*.Cu" "*.Mask")
-      (net 10 "/12") (pinfunction "Pin_6") (pintype "passive"))
-    (pad "7" thru_hole oval locked (at 0 15.24 90) (size 1.7 1.7) (drill 1) (layers "*.Cu" "*.Mask")
-      (net 14 "/*11") (pinfunction "Pin_7") (pintype "passive"))
-    (pad "8" thru_hole oval locked (at 0 17.78 90) (size 1.7 1.7) (drill 1) (layers "*.Cu" "*.Mask")
-      (net 15 "/*10") (pinfunction "Pin_8") (pintype "passive"))
-    (pad "9" thru_hole oval locked (at 0 20.32 90) (size 1.7 1.7) (drill 1) (layers "*.Cu" "*.Mask")
-      (net 16 "/*9") (pinfunction "Pin_9") (pintype "passive"))
-    (pad "10" thru_hole oval locked (at 0 22.86 90) (size 1.7 1.7) (drill 1) (layers "*.Cu" "*.Mask")
-      (net 12 "/8") (pinfunction "Pin_10") (pintype "passive"))
-    (model "${KICAD7_3DMODEL_DIR}/Connector_PinSocket_2.54mm.3dshapes/PinSocket_1x10_P2.54mm_Vertical.wrl"
-      (offset (xyz 0 0 0))
-      (scale (xyz 1 1 1))
-      (rotate (xyz 0 0 0))
-    )
-  )
   (footprint "Connector_PinSocket_2.54mm:PinSocket_1x08_P2.54mm_Vertical" locked (layer "F.Cu")
     (at 145.72 49.2 90)
@@
       (offset (xyz 0 0 0))
       (scale (xyz 1 1 1))
+      (rotate (xyz 0 0 0))
+    )
+  )
+  (footprint "Connector_PinHeader_2.54mm:PinHeader_1x10_P2.54mm_Vertical" (layer "B.Cu")
+    (at 118.796 49.2 -90)
+    (descr "Through hole straight pin header, 1x10, 2.54mm pitch, single row")
+    (tags "Through hole pin header THT 1x10 2.54mm single row")
+    (property "Sheetfile" "flipperbrain-shield.kicad_sch")
+    (property "Sheetname" "")
+    (property "ki_description" "Generic connector, single row, 01x10, script generated (kicad-library-utils/schlib/autogen/connector/)")
+    (property "ki_keywords" "connector")
+    (attr through_hole)
+    (fp_text reference "J2" (at 0 2.33 90) (layer "B.SilkS")
+        (effects (font (size 1 1) (thickness 0.15)) (justify mirror))
+    )
+    (fp_text value "Digital/PWM" (at 0 -25.19 90) (layer "B.Fab")
+        (effects (font (size 1 1) (thickness 0.15)) (justify mirror))
+    )
+    (fp_text user "${REFERENCE}" (at 0 -11.43 180) (layer "B.Fab")
+        (effects (font (size 1 1) (thickness 0.15)) (justify mirror))
+    )
+    (fp_line (start -1.33 -24.19) (end 1.33 -24.19)
+      (stroke (width 0.12) (type solid)) (layer "B.SilkS"))
+    (fp_line (start -1.33 -1.27) (end -1.33 -24.19)
+      (stroke (width 0.12) (type solid)) (layer "B.SilkS"))
+    (fp_line (start -1.33 -1.27) (end 1.33 -1.27)
+      (stroke (width 0.12) (type solid)) (layer "B.SilkS"))
+    (fp_line (start -1.33 0) (end -1.33 1.33)
+      (stroke (width 0.12) (type solid)) (layer "B.SilkS"))
+    (fp_line (start -1.33 1.33) (end 0 1.33)
+      (stroke (width 0.12) (type solid)) (layer "B.SilkS"))
+    (fp_line (start 1.33 -1.27) (end 1.33 -24.19)
+      (stroke (width 0.12) (type solid)) (layer "B.SilkS"))
+    (fp_line (start -1.8 -24.65) (end 1.8 -24.65)
+      (stroke (width 0.05) (type solid)) (layer "B.CrtYd"))
+    (fp_line (start -1.8 1.8) (end -1.8 -24.65)
+      (stroke (width 0.05) (type solid)) (layer "B.CrtYd"))
+    (fp_line (start 1.8 -24.65) (end 1.8 1.8)
+      (stroke (width 0.05) (type solid)) (layer "B.CrtYd"))
+    (fp_line (start 1.8 1.8) (end -1.8 1.8)
+      (stroke (width 0.05) (type solid)) (layer "B.CrtYd"))
+    (fp_line (start -1.27 -24.13) (end -1.27 0.635)
+      (stroke (width 0.1) (type solid)) (layer "B.Fab"))
+    (fp_line (start -1.27 0.635) (end -0.635 1.27)
+      (stroke (width 0.1) (type solid)) (layer "B.Fab"))
+    (fp_line (start -0.635 1.27) (end 1.27 1.27)
+      (stroke (width 0.1) (type solid)) (layer "B.Fab"))
+    (fp_line (start 1.27 -24.13) (end -1.27 -24.13)
+      (stroke (width 0.1) (type solid)) (layer "B.Fab"))
+    (fp_line (start 1.27 1.27) (end 1.27 -24.13)
+      (stroke (width 0.1) (type solid)) (layer "B.Fab"))
+    (pad "1" thru_hole rect (at 0 0 270) (size 1.7 1.7) (drill 1) (layers "*.Cu" "*.Mask")
+      (net 8 "/SCL{slash}A5") (pinfunction "Pin_1") (pintype "passive"))
+    (pad "2" thru_hole oval (at 0 -2.54 270) (size 1.7 1.7) (drill 1) (layers "*.Cu" "*.Mask")
+      (net 7 "/SDA{slash}A4") (pinfunction "Pin_2") (pintype "passive"))
+    (pad "3" thru_hole oval (at 0 -5.08 270) (size 1.7 1.7) (drill 1) (layers "*.Cu" "*.Mask")
+      (net 11 "/AREF") (pinfunction "Pin_3") (pintype "passive"))
+    (pad "4" thru_hole oval (at 0 -7.62 270) (size 1.7 1.7) (drill 1) (layers "*.Cu" "*.Mask")
+      (net 1 "GND") (pinfunction "Pin_4") (pintype "passive"))
+    (pad "5" thru_hole oval (at 0 -10.16 270) (size 1.7 1.7) (drill 1) (layers "*.Cu" "*.Mask")
+      (net 9 "/13") (pinfunction "Pin_5") (pintype "passive"))
+    (pad "6" thru_hole oval (at 0 -12.7 270) (size 1.7 1.7) (drill 1) (layers "*.Cu" "*.Mask")
+      (net 10 "/12") (pinfunction "Pin_6") (pintype "passive"))
+    (pad "7" thru_hole oval (at 0 -15.24 270) (size 1.7 1.7) (drill 1) (layers "*.Cu" "*.Mask")
+      (net 14 "/*11") (pinfunction "Pin_7") (pintype "passive"))
+    (pad "8" thru_hole oval (at 0 -17.78 270) (size 1.7 1.7) (drill 1) (layers "*.Cu" "*.Mask")
+      (net 15 "/*10") (pinfunction "Pin_8") (pintype "passive"))
+    (pad "9" thru_hole oval (at 0 -20.32 270) (size 1.7 1.7) (drill 1) (layers "*.Cu" "*.Mask")
+      (net 16 "/*9") (pinfunction "Pin_9") (pintype "passive"))
+    (pad "10" thru_hole oval (at 0 -22.86 270) (size 1.7 1.7) (drill 1) (layers "*.Cu" "*.Mask")
+      (net 12 "/8") (pinfunction "Pin_10") (pintype "passive"))
+    (model "${KICAD6_3DMODEL_DIR}/Connector_PinHeader_2.54mm.3dshapes/PinHeader_1x10_P2.54mm_Vertical.wrl"
+      (offset (xyz 0 0 0))
+      (scale (xyz 1 1 1))
