File: flipperbrain-shield/flipperbrain-shield/flipperbrain-shield.kicad_pcb (KiCad board)
At the start: 2 copper layers, 68.6 x 53.3 mm, 10 parts, among them J1 Power, J2 Digital/PWM, J3 Analog, J4 Digital/PWM

Commit message: nc
Parts:
- removed J4: Digital/PWM, Connector_PinSocket_2.54mm:PinSocket_1x08_P2.54mm_Vertical
- added J4-new1: Digital/PWM, Connector_PinHeader_2.54mm:PinHeader_1x08_P2.54mm_Vertical, B.Cu at (145.7, 49.2)
Changed lines of the file:
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@@
   (net 28 "Net-(D1-A)")
   (net 29 "unconnected-(J1-Pin_1-Pad1)")
-  (footprint "Connector_PinSocket_2.54mm:PinSocket_1x08_P2.54mm_Vertical" locked (layer "F.Cu")
-    (at 145.72 49.2 90)
-    (descr "Through hole straight socket strip, 1x08, 2.54mm pitch, single row (from Kicad 4.0.7), script generated")
-    (tags "Through hole socket strip THT 1x08 2.54mm single row")
-    (property "Sheetfile" "flipperbrain-shield.kicad_sch")
-    (property "Sheetname" "")
-    (property "ki_description" "Generic connector, single row, 01x08, script generated (kicad-library-utils/schlib/autogen/connector/)")
-    (property "ki_keywords" "connector")
-    (attr through_hole)
-    (fp_text reference "J4" (at 0 -2.77 90) (layer "F.SilkS") hide
-        (effects (font (size 1 1) (thickness 0.15)))
-    )
-    (fp_text value "Digital/PWM" (at 3.81 8.89 180) (layer "F.Fab")
-        (effects (font (size 1 1) (thickness 0.15)))
-    )
-    (fp_text user "${REFERENCE}" (at 3.81 0) (layer "F.Fab")
-        (effects (font (size 1 1) (thickness 0.15)))
-    )
-    (fp_line (start -1.33 1.27) (end -1.33 19.11)
-      (stroke (width 0.12) (type solid)) (layer "F.SilkS"))
-    (fp_line (start -1.33 1.27) (end 1.33 1.27)
-      (stroke (width 0.12) (type solid)) (layer "F.SilkS"))
-    (fp_line (start -1.33 19.11) (end 1.33 19.11)
-      (stroke (width 0.12) (type solid)) (layer "F.SilkS"))
-    (fp_line (start 0 -1.33) (end 1.33 -1.33)
-      (stroke (width 0.12) (type solid)) (layer "F.SilkS"))
-    (fp_line (start 1.33 -1.33) (end 1.33 0)
-      (stroke (width 0.12) (type solid)) (layer "F.SilkS"))
-    (fp_line (start 1.33 1.27) (end 1.33 19.11)
-      (stroke (width 0.12) (type solid)) (layer "F.SilkS"))
-    (fp_line (start -1.8 -1.8) (end 1.75 -1.8)
-      (stroke (width 0.05) (type solid)) (layer "F.CrtYd"))
-    (fp_line (start -1.8 19.55) (end -1.8 -1.8)
-      (stroke (width 0.05) (type solid)) (layer "F.CrtYd"))
-    (fp_line (start 1.75 -1.8) (end 1.75 19.55)
-      (stroke (width 0.05) (type solid)) (layer "F.CrtYd"))
-    (fp_line (start 1.75 19.55) (end -1.8 19.55)
-      (stroke (width 0.05) (type solid)) (layer "F.CrtYd"))
-    (fp_line (start -1.27 -1.27) (end 0.635 -1.27)
-      (stroke (width 0.1) (type solid)) (layer "F.Fab"))
-    (fp_line (start -1.27 19.05) (end -1.27 -1.27)
-      (stroke (width 0.1) (type solid)) (layer "F.Fab"))
-    (fp_line (start 0.635 -1.27) (end 1.27 -0.635)
-      (stroke (width 0.1) (type solid)) (layer "F.Fab"))
-    (fp_line (start 1.27 -0.635) (end 1.27 19.05)
-      (stroke (width 0.1) (type solid)) (layer "F.Fab"))
-    (fp_line (start 1.27 19.05) (end -1.27 19.05)
-      (stroke (width 0.1) (type solid)) (layer "F.Fab"))
-    (pad "1" thru_hole rect locked (at 0 0 90) (size 1.7 1.7) (drill 1) (layers "*.Cu" "*.Mask")
-      (net 13 "/7") (pinfunction "Pin_1") (pintype "passive"))
-    (pad "2" thru_hole oval locked (at 0 2.54 90) (size 1.7 1.7) (drill 1) (layers "*.Cu" "*.Mask")
-      (net 19 "/*6") (pinfunction "Pin_2") (pintype "passive"))
-    (pad "3" thru_hole oval locked (at 0 5.08 90) (size 1.7 1.7) (drill 1) (layers "*.Cu" "*.Mask")
-      (net 20 "/*5") (pinfunction "Pin_3") (pintype "passive"))
-    (pad "4" thru_hole oval locked (at 0 7.62 90) (size 1.7 1.7) (drill 1) (layers "*.Cu" "*.Mask")
-      (net 17 "/4") (pinfunction "Pin_4") (pintype "passive"))
-    (pad "5" thru_hole oval locked (at 0 10.16 90) (size 1.7 1.7) (drill 1) (layers "*.Cu" "*.Mask")
-      (net 22 "/*3") (pinfunction "Pin_5") (pintype "passive"))
-    (pad "6" thru_hole oval locked (at 0 12.7 90) (size 1.7 1.7) (drill 1) (layers "*.Cu" "*.Mask")
-      (net 18 "/2") (pinfunction "Pin_6") (pintype "passive"))
-    (pad "7" thru_hole oval locked (at 0 15.24 90) (size 1.7 1.7) (drill 1) (layers "*.Cu" "*.Mask")
-      (net 21 "/TX{slash}1") (pinfunction "Pin_7") (pintype "passive"))
-    (pad "8" thru_hole oval locked (at 0 17.78 90) (size 1.7 1.7) (drill 1) (layers "*.Cu" "*.Mask")
-      (net 23 "/RX{slash}0") (pinfunction "Pin_8") (pintype "passive"))
-    (model "${KICAD7_3DMODEL_DIR}/Connector_PinSocket_2.54mm.3dshapes/PinSocket_1x08_P2.54mm_Vertical.wrl"
-      (offset (xyz 0 0 0))
-      (scale (xyz 1 1 1))
-      (rotate (xyz 0 0 0))
-    )
-  )
   (footprint "Arduino_MountingHole:MountingHole_3.2mm" locked (layer "F.Cu")
     (at 115.24 49.2)
@@
       (offset (xyz 0 0 0))
       (scale (xyz 1 1 1))
+      (rotate (xyz 0 0 0))
+    )
+  )
+  (footprint "Connector_PinHeader_2.54mm:PinHeader_1x08_P2.54mm_Vertical" (layer "B.Cu")
+    (at 145.72 49.2 -90)
+    (descr "Through hole straight pin header, 1x08, 2.54mm pitch, single row")
+    (tags "Through hole pin header THT 1x08 2.54mm single row")
+    (property "Sheetfile" "flipperbrain-shield.kicad_sch")
+    (property "Sheetname" "")
+    (property "ki_description" "Generic connector, single row, 01x08, script generated (kicad-library-utils/schlib/autogen/connector/)")
+    (property "ki_keywords" "connector")
+    (attr through_hole)
+    (fp_text reference "J4-new1" (at 0 2.33 90) (layer "B.SilkS")
+        (effects (font (size 1 1) (thickness 0.15)) (justify mirror))
+    )
+    (fp_text value "Digital/PWM" (at 0 -20.11 90) (layer "B.Fab")
+        (effects (font (size 1 1) (thickness 0.15)) (justify mirror))
+    )
+    (fp_text user "${REFERENCE}" (at 0 -8.89 180) (layer "B.Fab")
+        (effects (font (size 1 1) (thickness 0.15)) (justify mirror))
+    )
+    (fp_line (start -1.33 -19.11) (end 1.33 -19.11)
+      (stroke (width 0.12) (type solid)) (layer "B.SilkS"))
+    (fp_line (start -1.33 -1.27) (end -1.33 -19.11)
+      (stroke (width 0.12) (type solid)) (layer "B.SilkS"))
+    (fp_line (start -1.33 -1.27) (end 1.33 -1.27)
+      (stroke (width 0.12) (type solid)) (layer "B.SilkS"))
+    (fp_line (start -1.33 0) (end -1.33 1.33)
+      (stroke (width 0.12) (type solid)) (layer "B.SilkS"))
+    (fp_line (start -1.33 1.33) (end 0 1.33)
+      (stroke (width 0.12) (type solid)) (layer "B.SilkS"))
+    (fp_line (start 1.33 -1.27) (end 1.33 -19.11)
+      (stroke (width 0.12) (type solid)) (layer "B.SilkS"))
+    (fp_line (start -1.8 -19.55) (end 1.8 -19.55)
+      (stroke (width 0.05) (type solid)) (layer "B.CrtYd"))
+    (fp_line (start -1.8 1.8) (end -1.8 -19.55)
+      (stroke (width 0.05) (type solid)) (layer "B.CrtYd"))
+    (fp_line (start 1.8 -19.55) (end 1.8 1.8)
+      (stroke (width 0.05) (type solid)) (layer "B.CrtYd"))
+    (fp_line (start 1.8 1.8) (end -1.8 1.8)
+      (stroke (width 0.05) (type solid)) (layer "B.CrtYd"))
+    (fp_line (start -1.27 -19.05) (end -1.27 0.635)
+      (stroke (width 0.1) (type solid)) (layer "B.Fab"))
+    (fp_line (start -1.27 0.635) (end -0.635 1.27)
+      (stroke (width 0.1) (type solid)) (layer "B.Fab"))
+    (fp_line (start -0.635 1.27) (end 1.27 1.27)
+      (stroke (width 0.1) (type solid)) (layer "B.Fab"))
+    (fp_line (start 1.27 -19.05) (end -1.27 -19.05)
+      (stroke (width 0.1) (type solid)) (layer "B.Fab"))
+    (fp_line (start 1.27 1.27) (end 1.27 -19.05)
+      (stroke (width 0.1) (type solid)) (layer "B.Fab"))
+    (pad "1" thru_hole rect (at 0 0 270) (size 1.7 1.7) (drill 1) (layers "*.Cu" "*.Mask")
+      (net 13 "/7") (pinfunction "Pin_1") (pintype "passive"))
+    (pad "2" thru_hole oval (at 0 -2.54 270) (size 1.7 1.7) (drill 1) (layers "*.Cu" "*.Mask")
+      (net 19 "/*6") (pinfunction "Pin_2") (pintype "passive"))
+    (pad "3" thru_hole oval (at 0 -5.08 270) (size 1.7 1.7) (drill 1) (layers "*.Cu" "*.Mask")
+      (net 20 "/*5") (pinfunction "Pin_3") (pintype "passive"))
+    (pad "4" thru_hole oval (at 0 -7.62 270) (size 1.7 1.7) (drill 1) (layers "*.Cu" "*.Mask")
+      (net 17 "/4") (pinfunction "Pin_4") (pintype "passive"))
+    (pad "5" thru_hole oval (at 0 -10.16 270) (size 1.7 1.7) (drill 1) (layers "*.Cu" "*.Mask")
+      (net 22 "/*3") (pinfunction "Pin_5") (pintype "passive"))
+    (pad "6" thru_hole oval (at 0 -12.7 270) (size 1.7 1.7) (drill 1) (layers "*.Cu" "*.Mask")
+      (net 18 "/2") (pinfunction "Pin_6") (pintype "passive"))
+    (pad "7" thru_hole oval (at 0 -15.24 270) (size 1.7 1.7) (drill 1) (layers "*.Cu" "*.Mask")
+      (net 21 "/TX{slash}1") (pinfunction "Pin_7") (pintype "passive"))
+    (pad "8" thru_hole oval (at 0 -17.78 270) (size 1.7 1.7) (drill 1) (layers "*.Cu" "*.Mask")
+      (net 23 "/RX{slash}0") (pinfunction "Pin_8") (pintype "passive"))
+    (model "${KICAD6_3DMODEL_DIR}/Connector_PinHeader_2.54mm.3dshapes/PinHeader_1x08_P2.54mm_Vertical.wrl"
+      (offset (xyz 0 0 0))
+      (scale (xyz 1 1 1))

Commit message: nc
Parts:
- removed MH3: MountingHole_3.2mm, Arduino_MountingHole:MountingHole_3.2mm
- added D2: LED, LED_THT:LED_D5.0mm, F.Cu at (123.3, 77.2)
- added D3: LED, LED_THT:LED_D5.0mm, F.Cu at (132.5, 77.2)
- added D4: LED, LED_THT:LED_D5.0mm, F.Cu at (141.6, 77.2)
- added D5: LED, LED_THT:LED_D5.0mm, F.Cu at (150.8, 77.2)
- added D6: LED, LED_THT:LED_D5.0mm, F.Cu at (159.9, 77.2)
- added J5: Screw_Terminal_01x06, TerminalBlock_Phoenix:TerminalBlock_Phoenix_PT-1,5-6-3.5-H_1x06_P3.50mm_Horizontal, F.Cu at (107.6, 73.2)
- added J6: Screw_Terminal_01x06, TerminalBlock_Phoenix:TerminalBlock_Phoenix_PT-1,5-6-3.5-H_1x06_P3.50mm_Horizontal, F.Cu at (107.5, 50.0)
- added R2: R, Resistor_THT:R_Axial_DIN0207_L6.3mm_D2.5mm_P10.16mm_Horizontal, F.Cu at (112.8, 84.7)
- added R3: R, Resistor_THT:R_Axial_DIN0207_L6.3mm_D2.5mm_P10.16mm_Horizontal, F.Cu at (143.2, 89.5)
- added R4: R, Resistor_THT:R_Axial_DIN0207_L6.3mm_D2.5mm_P10.16mm_Horizontal, F.Cu at (143.2, 84.7)
- added R5: R, Resistor_THT:R_Axial_DIN0207_L6.3mm_D2.5mm_P10.16mm_Horizontal, F.Cu at (163.3, 89.5)
- added R6: R, Resistor_THT:R_Axial_DIN0207_L6.3mm_D2.5mm_P10.16mm_Horizontal, F.Cu at (163.3, 84.7)
- added SW10: SW_Push, Button_Switch_THT:SW_PUSH_6mm, F.Cu at (131.6, 62.4)
- added SW11: SW_Push, Button_Switch_THT:SW_PUSH_6mm, F.Cu at (140.6, 62.4)
- added SW12: SW_Push, Button_Switch_THT:SW_PUSH_6mm, F.Cu at (149.7, 62.4)
- added SW13: SW_Push, Button_Switch_THT:SW_PUSH_6mm, F.Cu at (158.7, 62.4)
- added SW8: SW_Push, Button_Switch_THT:SW_PUSH_6mm, F.Cu at (113.6, 62.4)
- added SW9: SW_Push, Button_Switch_THT:SW_PUSH_6mm, F.Cu at (122.6, 62.4)
- moved R1 38.1 mm to (112.8, 89.5), turned to 0 degrees
- moved D1 37.0 mm to (114.2, 77.2), turned to 0 degrees
- renumbered J4-new1 to J4
Connections:
- net /SCL/A5 renamed A5
- net /SDA/A4 renamed A4
- J2 pad 10: /8 -> TD8
- J2 pad 5: /13 -> TD13
- J2 pad 6: /12 -> TD12
- J2 pad 7: /*11 -> TD11
- J2 pad 8: /*10 -> TD10
- J2 pad 9: /*9 -> TD9
- J3 pad 2: /A1 -> A1
- J3 pad 3: /A2 -> A2
- J3 pad 4: /A3 -> A3
Other:
- board text removed: "ICSP"

Commit message: nc
Parts:
- moved J5 7.05 mm to (105.2, 79.8)
- moved J6 2.33 mm to (105.2, 49.4)
Routing:
- net GND: track 0.00 -> 183.2 mm
- net A4: track 0.00 -> 122.9 mm
- net A5: track 0.00 -> 122.5 mm
- net TD13: track 0.00 -> 75.4 mm
- net TD11: track 0.00 -> 73.3 mm
- net TD12: track 0.00 -> 66.7 mm
- net A3: track 0.00 -> 66.1 mm
- net A0: track 0.00 -> 64.5 mm
- net TD9: track 0.00 -> 62.7 mm
- net TD8: track 0.00 -> 56.6 mm
- net TD10: track 0.00 -> 56.1 mm
- net A1: track 0.00 -> 56.0 mm
- net A2: track 0.00 -> 55.3 mm
- net Net-(D1-A): track 0.00 -> 14.9 mm
- net Net-(D4-A): track 0.00 -> 14.3 mm
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