File: flipperbrain-shield/flipperbrain-shield/flipperbrain-shield.kicad_pcb (KiCad board)
At the start: 2 copper layers, 68.6 x 53.3 mm, 27 parts, among them J1 Power, J2 Digital/PWM, J3 Analog, J4 Digital/PWM, J5 Screw_Terminal_01x06, J6 Screw_Terminal_01x06, SW10 SW_Push, SW11 SW_Push, SW12 SW_Push, SW13 SW_Push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

Commit message: nc
Parts:
- added G***: LOGO, LOGO, F.Cu at (130.5, 73.7)

Commit message: nc
Parts:
- added G002: LOGO, LOGO, F.Cu at (157.3, 93.7)
- renumbered G*** to G001
Routing:
- net TD12: track 66.7 -> 79.7 mm
- net TD9: track 62.7 -> 53.2 mm
- net TD10: track 56.1 -> 46.7 mm
- net TD13: track 75.4 -> 83.6 mm
- net TD8: track 56.6 -> 48.9 mm
- net TD11: track 73.3 -> 67.2 mm
- net A5: track 122.5 -> 128.2 mm
- net A4: track 122.9 -> 118.7 mm
- net GND: track 183.2 -> 180.3 mm
