File: flipperbrain-shield/flipperbrain-shield/flipperbrain-shield.kicad_pcb (KiCad board)
At the start: 2 copper layers, 68.6 x 53.3 mm, 24 parts, among them J1 Power, J2 Digital/PWM, J3 Analog, J4 Digital/PWM, J5 Screw_Terminal_01x06, J6 Screw_Terminal_01x06, SW10 SW_Push, SW11 SW_Push, SW12 SW_Push, SW13 SW_Push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

Commit message: nc
Parts:
- moved RN1 35.3 mm to (162.7, 86.9), turned to 180 degrees
Routing:
- net Net-(D6-K): track 40.1 -> 9.78 mm
- net A4: track 125.2 -> 107.5 mm
- net A1: track 84.1 -> 66.9 mm
- net Net-(D5-K): track 29.3 -> 12.5 mm
- net Net-(D3-K): track 11.0 -> 24.5 mm
- net Net-(D2-K): track 20.9 -> 31.1 mm
- net A0: track 64.7 -> 55.5 mm
- net GND: track 140.7 -> 147.0 mm
- net TD8: track 49.0 -> 54.5 mm
- net Net-(D4-K): track 15.1 -> 19.4 mm
- net Net-(D1-K): track 35.0 -> 38.7 mm
- net TD9: track 47.8 -> 44.7 mm
- net TD11: track 61.6 -> 64.3 mm
- net A3: track 83.3 -> 81.8 mm
- net A5: track 136.2 -> 137.5 mm
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