File: flipperbrain-shield/flipperbrain-shield/flipperbrain-shield.kicad_sch (KiCad schematic)
At the start: 6 parts, among them J1 Power, J2 Digital/PWM, J3 Analog, J4 Digital/PWM

Commit message: nc
Connections:
- net A0: now also R1.1; no longer D1.2 (A)
- net GND: now also D1.1 (K); no longer R1.2
- new net: D1.2 (A), R1.2
Other:
- moved on the sheet: D1, R1
Changed lines of the file:
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@@
     (stroke (width 0) (type solid))
+  )
+  (wire (pts (xy 120.65 52.07) (xy 120.65 53.34))
+    (stroke (width 0) (type default))
   )
   (wire (pts (xy 40.64 111.76) (xy 27.94 111.76))
@@
     (stroke (width 0) (type solid))
   )
+  (wire (pts (xy 120.65 60.96) (xy 120.65 63.5))
+    (stroke (width 0) (type default))
+  )
   (wire (pts (xy 62.23 62.23) (xy 74.93 62.23))
     (stroke (width 0) (type solid))
   )
+  (wire (pts (xy 120.65 41.91) (xy 120.65 44.45))
+    (stroke (width 0) (type default))
+  )
   (wire (pts (xy 62.23 46.99) (xy 74.93 46.99))
     (stroke (width 0) (type solid))
@@
     (effects (font (size 1.27 1.27)) (justify left bottom))
   )
-  (global_label "A0" (shape input) (at 120.65 59.69 90) (fields_autoplaced)
+  (global_label "A0" (shape input) (at 120.65 41.91 90) (fields_autoplaced)
     (effects (font (size 1.27 1.27)) (justify left))
-    (property "Intersheetrefs" "${INTERSHEET_REFS}" (at 120.65 54.391 90)
+    (property "Intersheetrefs" "${INTERSHEET_REFS}" (at 120.65 36.611 90)
       (effects (font (size 1.27 1.27)) (justify left) hide)
     )
   )
-  (global_label "GND" (shape input) (at 120.65 74.93 270) (fields_autoplaced)
+  (global_label "GND" (shape input) (at 120.65 63.5 270) (fields_autoplaced)
     (effects (font (size 1.27 1.27)) (justify right))
-    (property "Intersheetrefs" "${INTERSHEET_REFS}" (at 120.65 81.8014 90)
+    (property "Intersheetrefs" "${INTERSHEET_REFS}" (at 120.65 70.3714 90)
       (effects (font (size 1.27 1.27)) (justify right) hide)
     )
@@
     )
   )
-  (symbol (lib_id "Device:R") (at 120.65 71.12 0) (unit 1)
+  (symbol (lib_id "Device:R") (at 120.65 48.26 0) (unit 1)
     (in_bom yes) (on_board yes) (dnp no) (fields_autoplaced)
-    (property "Reference" "R1" (at 123.19 70.485 0)
+    (property "Reference" "R1" (at 123.19 47.625 0)
       (effects (font (size 1.27 1.27)) (justify left))
     )
-    (property "Value" "R" (at 123.19 73.025 0)
+    (property "Value" "R" (at 123.19 50.165 0)
       (effects (font (size 1.27 1.27)) (justify left))
     )
-    (property "Footprint" "Resistor_THT:R_Axial_DIN0207_L6.3mm_D2.5mm_P10.16mm_Horizontal" (at 118.872 71.12 90)
-      (effects (font (size 1.27 1.27)) hide)
-    )
-    (property "Datasheet" "~" (at 120.65 71.12 0)
+    (property "Footprint" "Resistor_THT:R_Axial_DIN0207_L6.3mm_D2.5mm_P10.16mm_Horizontal" (at 118.872 48.26 90)
+      (effects (font (size 1.27 1.27)) hide)
+    )
+    (property "Datasheet" "~" (at 120.65 48.26 0)
       (effects (font (size 1.27 1.27)) hide)
     )
@@
     )
   )
-  (symbol (lib_id "Device:LED") (at 120.65 63.5 90) (unit 1)
+  (symbol (lib_id "Device:LED") (at 120.65 57.15 90) (unit 1)
     (in_bom yes) (on_board yes) (dnp no) (fields_autoplaced)
-    (property "Reference" "D1" (at 124.46 64.4525 90)
+    (property "Reference" "D1" (at 124.46 58.1025 90)
       (effects (font (size 1.27 1.27)) (justify right))
     )
-    (property "Value" "LED" (at 124.46 66.9925 90)
+    (property "Value" "LED" (at 124.46 60.6425 90)
       (effects (font (size 1.27 1.27)) (justify right))
     )
-    (property "Footprint" "LED_THT:LED_D5.0mm" (at 120.65 63.5 0)
-      (effects (font (size 1.27 1.27)) hide)
-    )
-    (property "Datasheet" "~" (at 120.65 63.5 0)
-      (effects (font (size 1.27 1.27)) hide)
-    )
+    (property "Footprint" "LED_THT:LED_D5.0mm" (at 120.65 57.15 0)
+      (effects (font (size 1.27 1.27)) hide)
+    )
+    (property "Datasheet" "~" (at 120.65 57.15 0)
+      (effects (font (size 1.27 1.27)) hide)
+    )

Commit message: nc
Parts:
- J3: footprint Connector_PinSocket_2.54mm:PinSocket_1x06_P2.54mm_Vertical -> Connector_PinHeader_2.54mm:PinHeader_1x06_P2.54mm_Vertical
Changed lines of the file:
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@@
       (effects (font (size 1.27 1.27)))
     )
-    (property "Footprint" "Connector_PinSocket_2.54mm:PinSocket_1x06_P2.54mm_Vertical" (at 45.72 116.84 0)
+    (property "Footprint" "Connector_PinHeader_2.54mm:PinHeader_1x06_P2.54mm_Vertical" (at 45.72 116.84 0)
       (effects (font (size 1.27 1.27)) hide)
     )

Commit message: nc
Parts:
- added J1-new1: Power, Connector_PinHeader_2.54mm:PinHeader_1x08_P2.54mm_Vertical, symbol Connector_Generic:Conn_01x08
Connections:
- net +3V3: now also J1-new1.4 (Pin_4)
- net +5V: now also J1-new1.5 (Pin_5)
- net GND: now also J1-new1.6 (Pin_6), J1-new1.7 (Pin_7)
- net IOREF: now also J1-new1.2 (Pin_2)
- net VCC: now also J1-new1.8 (Pin_8)
- net ~{RESET}: now also J1-new1.3 (Pin_3)
- no-connect marks 1 -> 2
Other:
- moved on the sheet: J3

Commit message: nc
Parts:
- removed J1: Power, Connector_PinSocket_2.54mm:PinSocket_1x08_P2.54mm_Vertical, symbol Connector_Generic:Conn_01x08
- renumbered J1-new1 to J1
Connections:
- no-connect marks 2 -> 1
Changed lines of the file:
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@@
   (junction (at 33.02 99.06) (diameter 1.016) (color 0 0 0 0)
   )
-  (junction (at 31.75 46.99) (diameter 1.016) (color 0 0 0 0)
-  )
   (no_connect (at 35.56 83.82))
-  (no_connect (at 34.29 31.75))
   (wire (pts (xy 62.23 77.47) (xy 74.93 77.47))
     (stroke (width 0) (type solid))
@@
     (stroke (width 0) (type solid))
   )
-  (wire (pts (xy 31.75 44.45) (xy 31.75 46.99))
-    (stroke (width 0) (type solid))
-  )
   (wire (pts (xy 35.56 96.52) (xy 33.02 96.52))
     (stroke (width 0) (type solid))
@@
     (stroke (width 0) (type solid))
   )
-  (wire (pts (xy 31.75 46.99) (xy 31.75 52.07))
-    (stroke (width 0) (type solid))
-  )
-  (wire (pts (xy 31.75 39.37) (xy 34.29 39.37))
-    (stroke (width 0) (type solid))
-  )
-  (wire (pts (xy 29.21 41.91) (xy 34.29 41.91))
-    (stroke (width 0) (type solid))
-  )
-  (wire (pts (xy 29.21 26.67) (xy 29.21 41.91))
-    (stroke (width 0) (type solid))
-  )
   (wire (pts (xy 62.23 36.83) (xy 74.93 36.83))
-    (stroke (width 0) (type solid))
-  )
-  (wire (pts (xy 31.75 26.67) (xy 31.75 39.37))
     (stroke (width 0) (type solid))
   )
@@
     (stroke (width 0) (type solid))
   )
-  (wire (pts (xy 19.05 34.29) (xy 34.29 34.29))
-    (stroke (width 0) (type solid))
-  )
   (wire (pts (xy 33.02 99.06) (xy 33.02 104.14))
     (stroke (width 0) (type solid))
@@
     (stroke (width 0) (type solid))
   )
-  (wire (pts (xy 19.05 36.83) (xy 34.29 36.83))
-    (stroke (width 0) (type solid))
-  )
-  (wire (pts (xy 34.29 46.99) (xy 31.75 46.99))
-    (stroke (width 0) (type solid))
-  )
-  (wire (pts (xy 34.29 49.53) (xy 26.67 49.53))
-    (stroke (width 0) (type solid))
-  )
   (wire (pts (xy 153.67 115.57) (xy 166.37 115.57))
     (stroke (width 0) (type solid))
@@
     (stroke (width 0) (type solid))
   )
-  (wire (pts (xy 34.29 44.45) (xy 31.75 44.45))
-    (stroke (width 0) (type solid))
-  )
   (wire (pts (xy 62.23 41.91) (xy 74.93 41.91))
     (stroke (width 0) (type solid))
@@
     (stroke (width 0) (type solid))
   )
-  (wire (pts (xy 26.67 49.53) (xy 26.67 26.67))
-    (stroke (width 0) (type solid))
-  )
   (wire (pts (xy 166.37 123.19) (xy 153.67 123.19))
     (stroke (width 0) (type solid))
@@
     (effects (font (size 1.27 1.27)) (justify right bottom))
   )
-  (label "~{RESET}" (at 19.05 36.83 0) (fields_autoplaced)
-    (effects (font (size 1.27 1.27)) (justify left bottom))
-  )
   (label "*10" (at 74.93 44.45 180) (fields_autoplaced)
     (effects (font (size 1.27 1.27)) (justify right bottom))
@@
     (effects (font (size 1.27 1.27)) (justify right bottom))
   )
-  (label "Vin" (at 26.67 26.67 270) (fields_autoplaced)
-    (effects (font (size 1.27 1.27)) (justify right bottom))
-  )
   (label "*6" (at 74.93 62.23 180) (fields_autoplaced)
     (effects (font (size 1.27 1.27)) (justify right bottom))
@@
   (label "*5" (at 74.93 64.77 180) (fields_autoplaced)
     (effects (font (size 1.27 1.27)) (justify right bottom))
-  )
-  (label "IOREF" (at 19.05 34.29 0) (fields_autoplaced)
-    (effects (font (size 1.27 1.27)) (justify left bottom))
   )
   (label "SDA{slash}A4" (at 153.67 123.19 0) (fields_autoplaced)
@@
     (property "Intersheetrefs" "${INTERSHEET_REFS}" (at 148.371 113.03 0)
       (effects (font (size 1.27 1.27)) (justify right) hide)
-    )
-  )
-  (symbol (lib_id "Connector_Generic:Conn_01x08") (at 39.37 39.37 0) (unit 1)
-    (in_bom yes) (on_board yes) (dnp no)
-    (property "Reference" "J1" (at 39.37 29.21 0)
-      (effects (font (size 1.27 1.27)))
-    )
-    (property "Value" "Power" (at 41.91 39.37 90)
-      (effects (font (size 1.27 1.27)))
-    )
-    (property "Footprint" "Connector_PinSocket_2.54mm:PinSocket_1x08_P2.54mm_Vertical" (at 39.37 39.37 0)
-      (effects (font (size 1.27 1.27)) hide)
-    )
-    (property "Datasheet" "" (at 39.37 39.37 0)
-      (effects (font (size 1.27 1.27)))
-    )
-    (pin "1")
-    (pin "2")
-    (pin "3")
-    (pin "4")
-    (pin "5")
-    (pin "6")
-    (pin "7")
-    (pin "8")
-    (instances
-      (project "flipperbrain-shield"
-        (path "/e63e39d7-6ac0-4ffd-8aa3-1841a4541b55"
-          (reference "J1") (unit 1)
-        )
-      )
-    )
-  )
-  (symbol (lib_id "power:+3V3") (at 31.75 26.67 0) (unit 1)
-    (in_bom yes) (on_board yes) (dnp no)
-    (property "Reference" "#PWR03" (at 31.75 30.48 0)
-      (effects (font (size 1.27 1.27)) hide)
-    )
-    (property "Value" "+3.3V" (at 32.131 23.622 90)
-      (effects (font (size 1.27 1.27)) (justify left))
-    )
-    (property "Footprint" "" (at 31.75 26.67 0)
-      (effects (font (size 1.27 1.27)))
-    )
-    (property "Datasheet" "" (at 31.75 26.67 0)
-      (effects (font (size 1.27 1.27)))
-    )
-    (pin "1")
-    (instances
-      (project "flipperbrain-shield"
-        (path "/e63e39d7-6ac0-4ffd-8aa3-1841a4541b55"
-          (reference "#PWR03") (unit 1)
-        )
-      )
-    )
-  )
-  (symbol (lib_id "power:+5V") (at 29.21 26.67 0) (unit 1)
-    (in_bom yes) (on_board yes) (dnp no)
-    (property "Reference" "#PWR02" (at 29.21 30.48 0)
-      (effects (font (size 1.27 1.27)) hide)
-    )
-    (property "Value" "+5V" (at 29.5656 23.622 90)
-      (effects (font (size 1.27 1.27)) (justify left))
-    )
-    (property "Footprint" "" (at 29.21 26.67 0)
-      (effects (font (size 1.27 1.27)))
-    )
-    (property "Datasheet" "" (at 29.21 26.67 0)
-      (effects (font (size 1.27 1.27)))
-    )
-    (pin "1")
-    (instances
-      (project "flipperbrain-shield"
-        (path "/e63e39d7-6ac0-4ffd-8aa3-1841a4541b55"
-          (reference "#PWR02") (unit 1)
-        )
-      )
-    )
-  )
-  (symbol (lib_id "power:GND") (at 31.75 52.07 0) (unit 1)
-    (in_bom yes) (on_board yes) (dnp no)
-    (property "Reference" "#PWR04" (at 31.75 58.42 0)
-      (effects (font (size 1.27 1.27)) hide)
-    )
-    (property "Value" "GND" (at 31.75 55.88 0)
-      (effects (font (size 1.27 1.27)))
-    )
-    (property "Footprint" "" (at 31.75 52.07 0)
-      (effects (font (size 1.27 1.27)))
-    )
-    (property "Datasheet" "" (at 31.75 52.07 0)
-      (effects (font (size 1.27 1.27)))
-    )
-    (pin "1")
-    (instances
-      (project "flipperbrain-shield"
-        (path "/e63e39d7-6ac0-4ffd-8aa3-1841a4541b55"
-          (reference "#PWR04") (unit 1)
-        )
-      )
     )
   )
@@
   (symbol (lib_id "Connector_Generic:Conn_01x08") (at 40.64 91.44 0) (unit 1)
     (in_bom yes) (on_board yes) (dnp no)
-    (property "Reference" "J1-new1" (at 40.64 81.28 0)
+    (property "Reference" "J1" (at 40.64 81.28 0)
       (effects (font (size 1.27 1.27)))
     )
@@
       (project "flipperbrain-shield"
         (path "/e63e39d7-6ac0-4ffd-8aa3-1841a4541b55"
-          (reference "J1-new1") (unit 1)
+          (reference "J1") (unit 1)
         )
       )
@@
         )
       )
-    )
-  )
-  (symbol (lib_id "power:VCC") (at 26.67 26.67 0) (unit 1)
-    (in_bom yes) (on_board yes) (dnp no)
-    (property "Reference" "#PWR01" (at 26.67 30.48 0)
-      (effects (font (size 1.27 1.27)) hide)
-    )
-    (property "Value" "VCC" (at 27.051 23.622 90)
-      (effects (font (size 1.27 1.27)) (justify left))
-    )
-    (property "Footprint" "" (at 26.67 26.67 0)
-      (effects (font (size 1.27 1.27)) hide)
-    )
-    (property "Datasheet" "" (at 26.67 26.67 0)
-      (effects (font (size 1.27 1.27)) hide)
-    )
-    (pin "1")
-    (instances
-      (project "flipperbrain-shield"
-        (path "/e63e39d7-6ac0-4ffd-8aa3-1841a4541b55"
-          (reference "#PWR01") (unit 1)
-        )
-      )

Commit message: nc
Parts:
- J2: footprint Connector_PinSocket_2.54mm:PinSocket_1x10_P2.54mm_Vertical -> Connector_PinHeader_2.54mm:PinHeader_1x10_P2.54mm_Vertical

Commit message: nc
Parts:
- J4: footprint Connector_PinSocket_2.54mm:PinSocket_1x08_P2.54mm_Vertical -> Connector_PinHeader_2.54mm:PinHeader_1x08_P2.54mm_Vertical
Other:
- moved on the sheet: J2

Commit message: nc
Parts:
- added D2, D3, D4, D5, D6: LED, LED_THT:LED_D5.0mm, symbol Device:LED
- added J5, J6: Screw_Terminal_01x06, TerminalBlock_Phoenix:TerminalBlock_Phoenix_PT-1,5-6-3.5-H_1x06_P3.50mm_Horizontal, symbol Connector:Screw_Terminal_01x06
- added R2, R3, R4, R5, R6: R, Resistor_THT:R_Axial_DIN0207_L6.3mm_D2.5mm_P10.16mm_Horizontal, symbol Device:R
- added SW10, SW11, SW12, SW13, SW8, SW9: SW_Push, Button_Switch_THT:SW_PUSH_6mm, symbol Switch:SW_Push
Connections:
- net A0: now also J5.1 (Pin_1)
- net A1: now also J5.2 (Pin_2), R2.1
- net A2: now also J5.3 (Pin_3), R3.1
- net A3: now also J5.4 (Pin_4), R4.1
- net GND: now also D2.1 (K), D3.1 (K), D4.1 (K), D5.1 (K), D6.1 (K), SW10.1, SW11.1, SW12.1, SW13.1, SW8.1, SW9.1
- net *10 renamed TD10
- net TD10: now also J6.3 (Pin_3), SW10.2
- net *11 renamed TD11
- net TD11: now also J6.4 (Pin_4), SW11.2
- net *9 renamed TD9
- net TD9: now also J6.2 (Pin_2), SW9.2
- net 12 renamed TD12
- net TD12: now also J6.5 (Pin_5), SW12.2
- net 13 renamed TD13
- net TD13: now also J6.6 (Pin_6), SW13.2
- net 8 renamed TD8
- net TD8: now also J6.1 (Pin_1), SW8.2
- net SCL/A5 renamed A5
- net A5: now also J5.6 (Pin_6), R6.1
- net SDA/A4 renamed A4
- net A4: now also J5.5 (Pin_5), R5.1
- new net: D5.2 (A), R5.2
- new net: D3.2 (A), R3.2
- new net: D4.2 (A), R4.2
- new net: D6.2 (A), R6.2
- new net: D2.2 (A), R2.2
Other:
- moved on the sheet: D1, J2, J3, J4, R1

Commit message: nc
Parts:
- J5, J6: footprint TerminalBlock_Phoenix:TerminalBlock_Phoenix_PT-1,5-6-3.5-H_1x06_P3.50mm_Horizontal -> TerminalBlock_Phoenix:TerminalBlock_Phoenix_MPT-0,5-6-2.54_1x06_P2.54mm_Horizontal
Changed lines of the file:
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@@
       (effects (font (size 1.27 1.27)) (justify left))
     )
-    (property "Footprint" "TerminalBlock_Phoenix:TerminalBlock_Phoenix_PT-1,5-6-3.5-H_1x06_P3.50mm_Horizontal" (at 201.93 134.62 0)
+    (property "Footprint" "TerminalBlock_Phoenix:TerminalBlock_Phoenix_MPT-0,5-6-2.54_1x06_P2.54mm_Horizontal" (at 201.93 134.62 0)
       (effects (font (size 1.27 1.27)) hide)
     )
@@
       (effects (font (size 1.27 1.27)) (justify left))
     )
-    (property "Footprint" "TerminalBlock_Phoenix:TerminalBlock_Phoenix_PT-1,5-6-3.5-H_1x06_P3.50mm_Horizontal" (at 208.28 58.42 0)
-      (effects (font (size 1.27 1.27)) hide)
-    )
+    (property "Footprint" "TerminalBlock_Phoenix:TerminalBlock_Phoenix_MPT-0,5-6-2.54_1x06_P2.54mm_Horizontal" (at 208.28 58.42 0)
+      (effects (font (size 1.27 1.27)) hide)
+    )
